File: pcb/scot-motor-power.sch (KiCad schematic (older format))
At the start: 1 part

Commit message: WIP.
Parts:
- added C?: 2u2/35V, symbol Device:C
- added C? (x3): 1u/6.5V, symbol Device:C
- added C?: 10u/6.5V, symbol Device:C
- added C?: 1u/3V3, symbol Device:C
- added C?: 1u/5V, symbol Device:C
- added C?: 100n/3V3, symbol Device:C
- added D?: LED, symbol Device:LED
- added FB?: Ferrite_Bead_Small, symbol Device:Ferrite_Bead_Small
- added R?: 1K, symbol Device:R
- added R?: R, symbol Device:R
- added U?: MCP1703A-3302_SOT223, Package_TO_SOT_SMD:SOT-223-3_TabPin2, symbol Regulator_Linear:MCP1703A-3302_SOT223
- added U?: MCP1703A-5002_SOT223, Package_TO_SOT_SMD:SOT-223-3_TabPin2, symbol Regulator_Linear:MCP1703A-5002_SOT223
- added U?: TSR_1-2465, Converter_DCDC:Converter_DCDC_TRACO_TSR-1_THT, symbol Regulator_Switching:TSR_1-2465
Connections:
- net POWER_28V+: now reaches U?.1 (IN+), U?.2 (IN+), U?.3 (IN+)
- net POWER_28V+: now also U?.12 (VBUS), C?.1, U?.1 (Vin)
- net 3V3_MCU: now reaches U?.10 (VS)
- net 3V3_MCU: now also C?.1, C?.1, R?.2, U?.3 (VO)
- net GND: now reaches U?.11 (GND), U?.6 (GND)
- net GND: now also U?.4 (A1), U?.5 (A0), C?.2, C?.2, C?.2, C?.2, C?.2, C?.2, C?.2, C?.2, R?.2, U?.2 (GND), U?.2 (GND), U?.2 (GND)
- net MOTOR_28V+: now reaches U?.14 (IN-), U?.15 (IN-), U?.16 (IN-)
- net VI_ALERT: now reaches U?.7 (ALERT)
- net VI_ALERT: now also R?.1
- net VI_SDA: now reaches U?.8 (SDA)
- net VI_SCL: now reaches U?.9 (SCL)
- new net: C?.1, FB?.2, U?.3 (Vout)
- new net: D?.1 (K), R?.1
- new net 5V_CAN: C?.1, U?.3 (VO)
- new net VCC: C?.1, C?.1, C?.1, D?.2 (A), FB?.1, U?.1 (VI), U?.1 (VI)
Other:
- note added: "28VDC -> 6.5VDC Power Input"
- note added: "28VDC Motor Power Monitoring"
- note added: "6.5VDC -> 3.3VDC MCU"
- note added: "6.5VDC -> 5VDC CAN Transceiver"
- note added: "Power OK (Green)"
- moved on the sheet: U?

Commit message: WIP.
Parts:
- C16, C17, C18, C20, C21, C22, C23: renamed from C?; footprint (none) -> Capacitor_SMD:C_0603_1608Metric_Pad1.05x0.95mm_HandSolder
- C19: renamed from C?; footprint (none) -> Capacitor_SMD:C_0805_2012Metric_Pad1.15x1.40mm_HandSolder
- D5: renamed from D?; footprint (none) -> LED_SMD:LED_1210_3225Metric_Pad1.42x2.65mm_HandSolder
- FB2: renamed from FB?; footprint (none) -> Inductor_SMD:L_0805_2012Metric_Pad1.15x1.40mm_HandSolder
- R18: renamed from R?; footprint (none) -> Resistor_SMD:R_0603_1608Metric_Pad1.05x0.95mm_HandSolder
- R19: renamed from R?; footprint (none) -> Resistor_SMD:R_0805_2012Metric_Pad1.15x1.40mm_HandSolder
- gave numbers to parts that had none: 4
Connections:
- net MOTOR_28V+: now also U7.12 (VBUS)
- net POWER_28V+: no longer U7.12 (VBUS)
Changed lines of the file:
@@
 $EndDescr
 $Comp
-L Sensor:INA260 U?
+L Sensor:INA260 U7
 U 1 1 5E69848D
 P 4550 2950
-F 0 "U?" V 4504 2506 50  0000 R CNN
+F 0 "U7" V 4504 2506 50  0000 R CNN
 F 1 "INA260" V 4595 2506 50  0000 R CNN
 F 2 "Package_SO:TSSOP-16_4.4x5mm_P0.65mm" H 4550 2350 50  0001 C CNN
@@
 Text HLabel 3750 2500 0    50   Input ~ 0
 POWER_28V+
-Text HLabel 3750 2750 0    50   Input ~ 0
-POWER_28V-
-$Comp
-L Device:C C?
+$Comp
+L Device:C C17
 U 1 1 5E882EDF
 P 3450 5250
-F 0 "C?" H 3565 5296 50  0000 L CNN
+F 0 "C17" H 3565 5296 50  0000 L CNN
 F 1 "2u2/35V" H 3565 5205 50  0000 L CNN
-F 2 "" H 3488 5100 50  0001 C CNN
+F 2 "Capacitor_SMD:C_0603_1608Metric_Pad1.05x0.95mm_HandSolder" H 3488 5100 50  0001 C CNN
 F 3 "~" H 3450 5250 50  0001 C CNN
 	1    3450 5250
@@
 $EndComp
 $Comp
-L Device:C C?
+L Device:C C18
 U 1 1 5E883298
 P 4750 5250
-F 0 "C?" H 4865 5296 50  0000 L CNN
+F 0 "C18" H 4865 5296 50  0000 L CNN
 F 1 "1u/6.5V" H 4865 5205 50  0000 L CNN
-F 2 "" H 4788 5100 50  0001 C CNN
+F 2 "Capacitor_SMD:C_0603_1608Metric_Pad1.05x0.95mm_HandSolder" H 4788 5100 50  0001 C CNN
 F 3 "~" H 4750 5250 50  0001 C CNN
 	1    4750 5250
@@
 $EndComp
 $Comp
-L Device:Ferrite_Bead_Small FB?
+L Device:Ferrite_Bead_Small FB2
 U 1 1 5E884075
 P 5100 5100
-F 0 "FB?" V 4863 5100 50  0000 C CNN
+F 0 "FB2" V 4863 5100 50  0000 C CNN
 F 1 "Ferrite_Bead_Small" V 4954 5100 50  0000 C CNN
-F 2 "" V 5030 5100 50  0001 C CNN
+F 2 "Inductor_SMD:L_0805_2012Metric_Pad1.15x1.40mm_HandSolder" V 5030 5100 50  0001 C CNN
 F 3 "~" H 5100 5100 50  0001 C CNN
 	1    5100 5100
@@
 $EndComp
 $Comp
-L Device:C C?
+L Device:C C19
 U 1 1 5E88D35E
 P 5350 5250
-F 0 "C?" H 5465 5296 50  0000 L CNN
+F 0 "C19" H 5465 5296 50  0000 L CNN
 F 1 "10u/6.5V" H 5465 5205 50  0000 L CNN
-F 2 "" H 5388 5100 50  0001 C CNN
+F 2 "Capacitor_SMD:C_0805_2012Metric_Pad1.15x1.40mm_HandSolder" H 5388 5100 50  0001 C CNN
 F 3 "~" H 5350 5250 50  0001 C CNN
 	1    5350 5250
@@
 $EndComp
 $Comp
-L Regulator_Linear:MCP1703A-3302_SOT223 U?
+L Regulator_Linear:MCP1703A-3302_SOT223 U8
 U 1 1 5F0E873C
 P 8450 4300
-F 0 "U?" H 8450 4542 50  0000 C CNN
+F 0 "U8" H 8450 4542 50  0000 C CNN
 F 1 "MCP1703A-3302_SOT223" H 8450 4451 50  0000 C CNN
 F 2 "Package_TO_SOT_SMD:SOT-223-3_TabPin2" H 8450 4500 50  0001 C CNN
@@
 $EndComp
 $Comp
-L Device:C C?
+L Device:C C20
 U 1 1 5F0E8CBD
 P 7800 4450
-F 0 "C?" H 7915 4496 50  0000 L CNN
+F 0 "C20" H 7915 4496 50  0000 L CNN
 F 1 "1u/6.5V" H 7915 4405 50  0000 L CNN
-F 2 "" H 7838 4300 50  0001 C CNN
+F 2 "Capacitor_SMD:C_0603_1608Metric_Pad1.05x0.95mm_HandSolder" H 7838 4300 50  0001 C CNN
 F 3 "~" H 7800 4450 50  0001 C CNN
 	1    7800 4450
@@
 	7800 4300 8150 4300
 $Comp
-L Device:C C?
+L Device:C C22
 U 1 1 5F0E9FCA
 P 8800 4450
-F 0 "C?" H 8915 4496 50  0000 L CNN
+F 0 "C22" H 8915 4496 50  0000 L CNN
 F 1 "1u/3V3" H 8915 4405 50  0000 L CNN
-F 2 "" H 8838 4300 50  0001 C CNN
+F 2 "Capacitor_SMD:C_0603_1608Metric_Pad1.05x0.95mm_HandSolder" H 8838 4300 50  0001 C CNN
 F 3 "~" H 8800 4450 50  0001 C CNN
 	1    8800 4450
@@
 	4650 5100 4750 5100
 Connection ~ 4750 5100
-Wire Wire Line
-	6200 5400 6000 5400
 Connection ~ 4250 5400
 Wire Wire Line
@@
 	3450 5100 3850 5100
 $Comp
-L agg-kicad:VCC #PWR?
+L agg-kicad:VCC #PWR0130
 U 1 1 5F0ED075
 P 7800 4250
-F 0 "#PWR?" H 7800 4360 50  0001 L CNN
+F 0 "#PWR0130" H 7800 4360 50  0001 L CNN
 F 1 "VCC" H 7800 4373 50  0000 C CNN
 F 2 "" H 7800 4250 50  0001 C CNN
@@
 $EndComp
 $Comp
-L power:GND #PWR?
+L power:GND #PWR0131
 U 1 1 5F0ED86E
 P 7800 4650
-F 0 "#PWR?" H 7800 4400 50  0001 C CNN
+F 0 "#PWR0131" H 7800 4400 50  0001 C CNN
 F 1 "GND" H 7805 4477 50  0000 C CNN
 F 2 "" H 7800 4650 50  0001 C CNN
@@
 Connection ~ 7800 4300
 $Comp
-L agg-kicad:VCC #PWR?
+L agg-kicad:VCC #PWR0132
 U 1 1 5F0F5376
 P 5600 5050
-F 0 "#PWR?" H 5600 5160 50  0001 L CNN
+F 0 "#PWR0132" H 5600 5160 50  0001 L CNN
 F 1 "VCC" H 5600 5173 50  0000 C CNN
 F 2 "" H 5600 5050 50  0001 C CNN
@@
 Connection ~ 5350 5100
 $Comp
-L power:GND #PWR?
+L power:GND #PWR0133
 U 1 1 5F0F634F
 P 4250 5400
-F 0 "#PWR?" H 4250 5150 50  0001 C CNN
+F 0 "#PWR0133" H 4250 5150 50  0001 C CNN
 F 1 "GND" H 4255 5227 50  0000 C CNN
 F 2 "" H 4250 5400 50  0001 C CNN
@@
 Connection ~ 8800 4300
 $Comp
-L Device:C C?
+L Device:C C21
 U 1 1 5F111717
 P 7850 5900
-F 0 "C?" H 7965 5946 50  0000 L CNN
+F 0 "C21" H 7965 5946 50  0000 L CNN
 F 1 "1u/6.5V" H 7965 5855 50  0000 L CNN
-F 2 "" H 7888 5750 50  0001 C CNN
+F 2 "Capacitor_SMD:C_0603_1608Metric_Pad1.05x0.95mm_HandSolder" H 7888 5750 50  0001 C CNN
 F 3 "~" H 7850 5900 50  0001 C CNN
 	1    7850 5900
@@
 	7850 5750 8200 5750
 $Comp
-L Device:C C?
+L Device:C C23
 U 1 1 5F111723
 P 8850 5900
-F 0 "C?" H 8965 5946 50  0000 L CNN
+F 0 "C23" H 8965 5946 50  0000 L CNN
 F 1 "1u/5V" H 8965 5855 50  0000 L CNN
-F 2 "" H 8888 5750 50  0001 C CNN
+F 2 "Capacitor_SMD:C_0603_1608Metric_Pad1.05x0.95mm_HandSolder" H 8888 5750 50  0001 C CNN
 F 3 "~" H 8850 5900 50  0001 C CNN
 	1    8850 5900
@@
 	8850 5750 8800 5750
 $Comp
-L agg-kicad:VCC #PWR?
+L agg-kicad:VCC #PWR0134
 U 1 1 5F111730
 P 7850 5700
-F 0 "#PWR?" H 7850 5810 50  0001 L CNN
+F 0 "#PWR0134" H 7850 5810 50  0001 L CNN
 F 1 "VCC" H 7850 5823 50  0000 C CNN
 F 2 "" H 7850 5700 50  0001 C CNN
@@
 $EndComp
 $Comp
-L power:GND #PWR?
+L power:GND #PWR0135
 U 1 1 5F11173A
 P 7850 6100
-F 0 "#PWR?" H 7850 5850 50  0001 C CNN
+F 0 "#PWR0135" H 7850 5850 50  0001 C CNN
 F 1 "GND" H 7855 5927 50  0000 C CNN
 F 2 "" H 7850 6100 50  0001 C CNN
@@
 	7850 6050 8500 6050
 $Comp
-L Regulator_Linear:MCP1703A-5002_SOT223 U?
+L Regulator_Linear:MCP1703A-5002_SOT223 U9
 U 1 1 5F1147A2
 P 8500 5750
-F 0 "U?" H 8500 5992 50  0000 C CNN
+F 0 "U9" H 8500 5992 50  0000 C CNN
 F 1 "MCP1703A-5002_SOT223" H 8500 5901 50  0000 C CNN
 F 2 "Package_TO_SOT_SMD:SOT-223-3_TabPin2" H 8500 5950 50  0001 C CNN
@@
 	8500 6050 8850 6050
 $Comp
-L Regulator_Switching:TSR_1-2465 U?
+L Regulator_Switching:TSR_1-2465 U6
 U 1 1 5F1169B0
 P 4250 5200
-F 0 "U?" H 4250 5567 50  0000 C CNN
+F 0 "U6" H 4250 5567 50  0000 C CNN
 F 1 "TSR_1-2465" H 4250 5476 50  0000 C CNN
 F 2 "Converter_DCDC:Converter_DCDC_TRACO_TSR-1_THT" H 4250 5050 50  0001 L CIN
@@
 Connection ~ 4750 3400
 $Comp
-L power:GND #PWR?
+L power:GND #PWR0136
 U 1 1 5F11D008
 P 5350 2950
-F 0 "#PWR?" H 5350 2700 50  0001 C CNN
+F 0 "#PWR0136" H 5350 2700 50  0001 C CNN
 F 1 "GND" H 5355 2777 50  0000 C CNN
 F 2 "" H 5350 2950 50  0001 C CNN
@@
 	5350 2950 4950 2950
 Connection ~ 4950 2950
-Text HLabel 5350 2750 2    50   Input ~ 0
-MOTOR_28V-
 Text HLabel 5350 2500 2    50   Input ~ 0
 MOTOR_28V+
 Wire Wire Line
-	5350 2750 4950 2750
-Wire Wire Line
-	4950 2750 4950 2950
-Wire Wire Line
 	5350 2500 4750 2500
 Wire Wire Line
@@
 	4450 2550 4450 2500
 Wire Wire Line
-	4450 2500 4350 2500
-Wire Wire Line
 	4350 2500 4350 2550
 Wire Wire Line
 	4350 2500 3750 2500
-Connection ~ 4350 2500
-$Comp
-L power:GND #PWR?
-U 1 1 5F12103E
-P 3850 2750
-F 0 "#PWR?" H 3850 2500 50  0001 C CNN
-F 1 "GND" H 3855 2577 50  0000 C CNN
-F 2 "" H 3850 2750 50  0001 C CNN
-F 3 "" H 3850 2750 50  0001 C CNN
-	1    3850 2750
-	1    0    0    -1
-$EndComp
-Wire Wire Line
-	3850 2750 3750 2750
 Text HLabel 3400 3050 0    50   Input ~ 0
 3V3_MCU
 $Comp
-L Device:C C?
+L Device:C C16
 U 1 1 5F123658
 P 3450 3200
-F 0 "C?" H 3565 3246 50  0000 L CNN
+F 0 "C16" H 3565 3246 50  0000 L CNN
 F 1 "100n/3V3" H 3565 3155 50  0000 L CNN
-F 2 "" H 3488 3050 50  0001 C CNN
+F 2 "Capacitor_SMD:C_0603_1608Metric_Pad1.05x0.95mm_HandSolder" H 3488 3050 50  0001 C CNN
 F 3 "~" H 3450 3200 50  0001 C CNN
 	1    3450 3200
@@
 $EndComp
 $Comp
-L Device:R R?
+L Device:R R18
 U 1 1 5F1256CC
 P 4050 3200
-F 0 "R?" H 3980 3154 50  0000 R CNN
+F 0 "R18" H 3980 3154 50  0000 R CNN
 F 1 "1K" H 3980 3245 50  0000 R CNN
-F 2 "" V 3980 3200 50  0001 C CNN
+F 2 "Resistor_SMD:R_0603_1608Metric_Pad1.05x0.95mm_HandSolder" V 3980 3200 50  0001 C CNN
 F 3 "~" H 4050 3200 50  0001 C CNN
 	1    4050 3200
@@
 	3450 3050 3400 3050
 $Comp
-L power:GND #PWR?
+L power:GND #PWR0137
 U 1 1 5F129CB1
 P 3450 3350
-F 0 "#PWR?" H 3450 3100 50  0001 C CNN
+F 0 "#PWR0137" H 3450 3100 50  0001 C CNN
 F 1 "GND" H 3455 3177 50  0000 C CNN
 F 2 "" H 3450 3350 50  0001 C CNN
@@
 Text HLabel 3400 5100 0    50   Input ~ 0
 POWER_28V+
-Text HLabel 3400 5400 0    50   Input ~ 0
-POWER_28V-
 Wire Wire Line
 	3450 5100 3400 5100
 Connection ~ 3450 5100
-Wire Wire Line
-	3450 5400 3400 5400
-Connection ~ 3450 5400
-Text HLabel 6200 5400 2    50   Input ~ 0
-LV_GND
 Connection ~ 5350 5400
 Wire Wire Line
@@
 28VDC Motor Power Monitoring
 $Comp
-L Device:LED D?
+L Device:LED D5
 U 1 1 5F14C759
 P 5850 5100
-F 0 "D?" H 5843 4845 50  0000 C CNN
+F 0 "D5" H 5843 4845 50  0000 C CNN
 F 1 "LED" H 5843 4936 50  0000 C CNN
-F 2 "" H 5850 5100 50  0001 C CNN
+F 2 "LED_SMD:LED_1210_3225Metric_Pad1.42x2.65mm_HandSolder" H 5850 5100 50  0001 C CNN
 F 3 "~" H 5850 5100 50  0001 C CNN
 	1    5850 5100
@@
 $EndComp
 $Comp
-L Device:R R?
+L Device:R R19
 U 1 1 5F14D886
 P 6000 5250
-F 0 "R?" H 6070 5296 50  0000 L CNN
+F 0 "R19" H 6070 5296 50  0000 L CNN
 F 1 "R" H 6070 5205 50  0000 L CNN
-F 2 "" V 5930 5250 50  0001 C CNN
+F 2 "Resistor_SMD:R_0805_2012Metric_Pad1.15x1.40mm_HandSolder" V 5930 5250 50  0001 C CNN
 F 3 "~" H 6000 5250 50  0001 C CNN
 	1    6000 5250
 	1    0    0    -1
 $EndComp
-Connection ~ 6000 5400
 Wire Wire Line
 	6000 5400 5350 5400
@@
 Wire Notes Line
 	6200 2100 2800 2100
+Wire Wire Line
+	4750 2500 4450 2500
+Connection ~ 4750 2500
 $EndSCHEMATC
