File: pcb/scot-motor-mcu.sch (KiCad schematic (older format))
At the start: 51 parts, among them IC2 STM32F0xxKxTx, IC3 NCV8450A, J8 Conn_01x03_Male, P1 SWD, Q1 BC817, U1 LTV-357T, U10 74AHC1G08, U2 74HC00, U3 LTV-357T, U4 LTV-357T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

Commit message: pcb: Fix MCU xtal load capacitors.
Parts:
- C6, C7: value 12p -> 8p
Other:
- note added: "Xtal Load: 18pF\nBoard + Pin: 10pF"
Changed lines of the file:
@@
 P 2250 3550
 F 0 "C6" V 1998 3550 50  0000 C CNN
-F 1 "12p" V 2089 3550 50  0000 C CNN
+F 1 "8p" V 2089 3550 50  0000 C CNN
 F 2 "Capacitor_SMD:C_0603_1608Metric_Pad1.05x0.95mm_HandSolder" H 2288 3400 50  0001 C CNN
 F 3 "~" H 2250 3550 50  0001 C CNN
@@
 P 2250 4050
 F 0 "C7" V 1998 4050 50  0000 C CNN
-F 1 "12p" V 2089 4050 50  0000 C CNN
+F 1 "8p" V 2089 4050 50  0000 C CNN
 F 2 "Capacitor_SMD:C_0603_1608Metric_Pad1.05x0.95mm_HandSolder" H 2288 3900 50  0001 C CNN
 F 3 "~" H 2250 4050 50  0001 C CNN
@@
 Wire Wire Line
 	9000 1900 9000 1600
+Text Notes 1250 3900 0    50   ~ 0
+Xtal Load: 18pF\nBoard + Pin: 10pF
 $EndSCHEMATC
